File: deviantlcd.brd (EAGLE design)
At the start: 86.4 x 54.6 mm, 83 parts

Commit message: BOM done.
Parts:
- LED1: value (none) -> blue
- LED2: value (none) -> green
- R10, R11, R12, R13, R15, R16, R17, R18, R19, R21, R22, R23, R24, R26, R27, R28, R29, R30, R32, R35, R36, R37, R38, R39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: value (none) -> 33
- R33, R45, R46, R47, R48: value 4.75K -> 150
- R34: value 4.75K -> 50
