File: deviantlcd.sch (EAGLE design)
At the start: 83 parts

Commit message: BOM done.
Parts:
- C1, C10, C11, C2, C3, C4, C5, C7, C8, C9: MPN (none) -> VJ0603V104ZXXCW1BC
- C17, C19: MPN (none) -> C1608X7R1C105K
- C18: MPN (none) -> VJ0603Y103KXACW1BC
- C6: MPN (none) -> LMK107BBJ106MALT
- LED1: value (none) -> blue; MPN (none) -> HT-193NB-5589
- LED2: value (none) -> green; MPN (none) -> LG Q971-KN-1
- P6: MPN (none) -> TSHC-105-D-03-255-GT-LF
- P8, P9: MPN (none) -> TSHC-123-D-03-255-GT-LF
- R1, R3: MPN (none) -> RK73B1JTTDD562J
- R10, R11, R12, R13, R15, R16, R17, R18, R19, R21, R22, R23, R24, R26, R27, R29, R30, R32, R35, R36, R37, R38, R39, R40, R41, R56, R57, R58, R8: value (none) -> 33; MPN (none) -> CR0402-JW-330GLF
- R2, R4, R5, R7: MPN (none) -> CR0603-FX-4751GLF
- R28: value (none) -> 33
- R33, R45, R46, R47, R48: value 4.75K -> 150; MPN (none) -> 302-150-RC
- R34: value 4.75K -> 50; MPN (none) -> 302-49.9-RC
- R42, R9: MPN (none) -> WR06X1002FTL
- R43, R44, R49, R50, R51, R52, R53, R54: MPN (none) -> ERJ-2GE0R00X
- S1: MPN (none) -> 219-2MST
- SV1: MPN (none) -> NPTC132KFMS-RC
- U$1: MPN (none) -> CAT24C256WI-GT3
- U$10: MPN (none) -> LP3985IM5-2.8/NOPB
- U$3: MPN (none) -> SN74LVCH16T245DGGR
- U$4: MPN (none) -> NHD-2.4-240320SF-CTXI#-T1
- U$7, U$8: MPN (none) -> SN74LVC1T45DBVR
Other:
- note added: "DeviantLCD"
- note removed: "Cape Name"
